File: revC/cad/eagle/warp-revC.sch (EAGLE design)
At the start: 13 parts, among them J2 QIIC connector, J3 QIIC connector, J4 DF40FC-20DP-0.4V(51), J5 CORTEX_DEBUG_SMD, U1 MAX40200, U2 MAX40200

Commit message: Rerouted FPGA
Connections:
- net GND: now also U2.IOB_25B_G3, U2.RGB1
- net VCC: now also U2.IOB_12A_G4_CDONE, U2.IOB_2A; no longer U2.VCCIO_0
- net VCC_1V2: now also U2.IOB_10A, U2.IOT_46B_G0, U2.VCCIO_0
Changed lines of the file:
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@@
 <part name="C7" library="SparkFun-Passives" deviceset="CAP" device="0402-CAP" value="0.1uF"/>
 <part name="C6" library="SparkFun-Passives" deviceset="CAP" device="0402-CAP" value="10uF"/>
+<part name="GND4" library="supply1" library_urn="urn:adsk.eagle:library:371" deviceset="GND" device=""/>
+<part name="SUPPLY1" library="SparkFun-PowerSymbols" deviceset="VCC" device=""/>
+<part name="SUPPLY2" library="SparkFun-PowerSymbols" deviceset="VCC" device=""/>
+<part name="GND5" library="supply1" library_urn="urn:adsk.eagle:library:371" deviceset="GND" device=""/>
 </parts>
 <sheets>
@@
 <attribute name="VALUE" x="195.58" y="175.26" size="1.778" layer="96" rot="R90"/>
 </instance>
-<instance part="P+4" gate="VCC" x="208.28" y="116.84" smashed="yes">
-<attribute name="VALUE" x="205.74" y="114.3" size="1.778" layer="96" rot="R90"/>
+<instance part="P+4" gate="VCC" x="205.74" y="119.38" smashed="yes">
+<attribute name="VALUE" x="203.2" y="116.84" size="1.778" layer="96" rot="R90"/>
 </instance>
 <instance part="P+5" gate="VCC" x="317.5" y="124.46" smashed="yes">
@@
 <attribute name="NAME" x="313.944" y="114.681" size="1.778" layer="95"/>
 <attribute name="VALUE" x="313.944" y="109.601" size="1.778" layer="96"/>
+</instance>
+<instance part="GND4" gate="1" x="193.04" y="116.84" smashed="yes">
+<attribute name="VALUE" x="190.5" y="114.3" size="1.778" layer="96"/>
+</instance>
+<instance part="SUPPLY1" gate="G$1" x="195.58" y="144.78" smashed="yes">
+<attribute name="VALUE" x="195.58" y="147.574" size="1.778" layer="96" align="bottom-center"/>
+</instance>
+<instance part="SUPPLY2" gate="G$1" x="190.5" y="63.5" smashed="yes">
+<attribute name="VALUE" x="190.5" y="66.294" size="1.778" layer="96" align="bottom-center"/>
+</instance>
+<instance part="GND5" gate="1" x="198.12" y="76.2" smashed="yes">
+<attribute name="VALUE" x="195.58" y="73.66" size="1.778" layer="96"/>
 </instance>
 </instances>
@@
 <wire x1="149.86" y1="198.12" x2="203.2" y2="198.12" width="0.1524" layer="91"/>
 <label x="190.5" y="198.12" size="1.778" layer="95"/>
-<pinref part="U2" gate="G$1" pin="VCC"/>
-<wire x1="203.2" y1="154.94" x2="175.26" y2="154.94" width="0.1524" layer="91"/>
-<label x="177.8" y="154.94" size="1.778" layer="95"/>
-<wire x1="203.2" y1="154.94" x2="203.2" y2="180.34" width="0.1524" layer="91"/>
+<wire x1="203.2" y1="165.1" x2="203.2" y2="180.34" width="0.1524" layer="91"/>
 <wire x1="203.2" y1="180.34" x2="203.2" y2="198.12" width="0.1524" layer="91"/>
 <pinref part="TP1" gate="G$1" pin="PP"/>
@@
 <pinref part="C2" gate="G$1" pin="1"/>
 <pinref part="C3" gate="G$1" pin="1"/>
+<pinref part="U2" gate="G$1" pin="VCCIO_0"/>
+<wire x1="175.26" y1="165.1" x2="203.2" y2="165.1" width="0.1524" layer="91"/>
+<label x="177.8" y="165.1" size="1.778" layer="95"/>
+</segment>
+<segment>
+<pinref part="U2" gate="G$1" pin="VCC"/>
+<wire x1="190.5" y1="154.94" x2="175.26" y2="154.94" width="0.1524" layer="91"/>
+<label x="177.8" y="154.94" size="1.778" layer="95"/>
+</segment>
+<segment>
+<pinref part="U2" gate="G$1" pin="IOB_10A"/>
+<wire x1="175.26" y1="144.78" x2="190.5" y2="144.78" width="0.1524" layer="91"/>
+<label x="177.8" y="144.78" size="1.778" layer="95"/>
+</segment>
+<segment>
+<pinref part="U2" gate="G$1" pin="IOT_46B_G0"/>
+<wire x1="175.26" y1="76.2" x2="187.96" y2="76.2" width="0.1524" layer="91"/>
+<label x="177.8" y="76.2" size="1.778" layer="95"/>
 </segment>
 </net>
@@
 <pinref part="C4" gate="G$1" pin="1"/>
 <pinref part="C5" gate="G$1" pin="1"/>
+<label x="177.8" y="134.62" size="1.778" layer="95"/>
 </segment>
 </net>
@@
 <pinref part="C2" gate="G$1" pin="2"/>
 </segment>
+<segment>
+<pinref part="GND4" gate="1" pin="GND"/>
+<wire x1="193.04" y1="119.38" x2="193.04" y2="121.92" width="0.1524" layer="91"/>
+<pinref part="U2" gate="G$1" pin="IOB_25B_G3"/>
+<wire x1="175.26" y1="114.3" x2="185.42" y2="114.3" width="0.1524" layer="91"/>
+<wire x1="185.42" y1="114.3" x2="185.42" y2="121.92" width="0.1524" layer="91"/>
+<wire x1="193.04" y1="121.92" x2="185.42" y2="121.92" width="0.1524" layer="91"/>
+<label x="177.8" y="114.3" size="1.778" layer="95"/>
+</segment>
+<segment>
+<pinref part="U2" gate="G$1" pin="RGB1"/>
+<wire x1="175.26" y1="71.12" x2="190.5" y2="71.12" width="0.1524" layer="91"/>
+<wire x1="190.5" y1="71.12" x2="190.5" y2="78.74" width="0.1524" layer="91"/>
+<wire x1="190.5" y1="78.74" x2="198.12" y2="78.74" width="0.1524" layer="91"/>
+<pinref part="GND5" gate="1" pin="GND"/>
+<label x="177.8" y="71.12" size="1.778" layer="95"/>
+</segment>
 </net>
 <net name="CRESET_B" class="0">
@@
 <net name="VCC" class="0">
 <segment>
-<label x="177.8" y="165.1" size="1.778" layer="95"/>
-<pinref part="U2" gate="G$1" pin="VCCIO_0"/>
-<wire x1="175.26" y1="165.1" x2="198.12" y2="165.1" width="0.1524" layer="91"/>
-<wire x1="198.12" y1="165.1" x2="198.12" y2="167.64" width="0.1524" layer="91"/>
 <label x="177.8" y="160.02" size="1.778" layer="95"/>
 <pinref part="U2" gate="G$1" pin="VCCIO_2"/>
 <wire x1="198.12" y1="167.64" x2="198.12" y2="175.26" width="0.1524" layer="91"/>
 <wire x1="175.26" y1="160.02" x2="198.12" y2="160.02" width="0.1524" layer="91"/>
-<wire x1="198.12" y1="160.02" x2="198.12" y2="165.1" width="0.1524" layer="91"/>
-<junction x="198.12" y="165.1"/>
+<wire x1="198.12" y1="160.02" x2="198.12" y2="167.64" width="0.1524" layer="91"/>
 <pinref part="VCC" gate="VCC" pin="VCC"/>
 <wire x1="175.26" y1="167.64" x2="198.12" y2="167.64" width="0.1524" layer="91"/>
@@
 <label x="177.8" y="111.76" size="1.778" layer="95"/>
 <pinref part="U2" gate="G$1" pin="SPI_VCCIO1"/>
-<wire x1="175.26" y1="111.76" x2="208.28" y2="111.76" width="0.1524" layer="91"/>
-<wire x1="208.28" y1="111.76" x2="208.28" y2="114.3" width="0.1524" layer="91"/>
+<wire x1="175.26" y1="111.76" x2="205.74" y2="111.76" width="0.1524" layer="91"/>
+<wire x1="205.74" y1="111.76" x2="205.74" y2="116.84" width="0.1524" layer="91"/>
 <pinref part="P+4" gate="VCC" pin="VCC"/>
 </segment>
@@
 <pinref part="P+2" gate="VCC" pin="VCC"/>
 </segment>
-</net>
+<segment>
+<pinref part="U2" gate="G$1" pin="IOB_12A_G4_CDONE"/>
+<wire x1="175.26" y1="139.7" x2="195.58" y2="139.7" width="0.1524" layer="91"/>
+<wire x1="195.58" y1="139.7" x2="195.58" y2="144.78" width="0.1524" layer="91"/>
+<pinref part="SUPPLY1" gate="G$1" pin="VCC"/>
+<label x="177.8" y="139.7" size="1.778" layer="95"/>
+</segment>
+<segment>
+<pinref part="U2" gate="G$1" pin="IOB_2A"/>
+<wire x1="175.26" y1="60.96" x2="190.5" y2="60.96" width="0.1524" layer="91"/>
+<pinref part="SUPPLY2" gate="G$1" pin="VCC"/>
+<wire x1="190.5" y1="60.96" x2="190.5" y2="63.5" width="0.1524" layer="91"/>
+<label x="177.8" y="60.96" size="1.778" layer="95"/>
+</segment>
+</net>
